Commit message: some tyops

File: urdf/bike.urdf (robot description, URDF)
Before this commit: robot frame, 5 links, 4 joints
Links:
- link backWheelLink: geometry collision mesh filename=package://ecn_mobile_control/urdf/files/wheel_scaled.stl; visual mesh filename=package://ecn_mobile_control/urdf/files/wheel_scaled.stl
- link frameLink: geometry collision mesh filename=package://ecn_mobile_control/urdf/files/frame_scaled_left.s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; collision mesh filename=package://ecn_mobile_control/urdf/files/frame_scaled_right.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
- link frontWheelLink: geometry collision mesh filename=package://ecn_mobile_control/urdf/files/wheel_scaled.stl; visual mesh filename=package://ecn_mobile_control/urdf/files/wheel_scaled.stl
- link handlebarLink: geometry collision mesh filename=package://ecn_mobile_control/urdf/files/handlebar_scaled.stl; visual mesh filename=package://ecn_mobile_control/urdf/files/handlebar_scaled.stl

Commit message: add actual carrot for carrot-based control

File: urdf/bike.urdf (robot description, URDF)
Before this commit: robot frame, 5 links, 4 joints
Links:
- added link carrot; visual mesh filename=package://ecn_mobile_control/urdf/carrot/carrot.dae scale=0.003 0.003 0.003
- added link carrot_disable
Joints:
- added joint carrot: type prismatic, parent carrot_disable, child carrot, axis 1 0 0, limit lower=-100 upper=100 effort=-1 velocity=10
- added joint carrot_disable: type prismatic, parent handlebarLink, child carrot_disable, origin xyz=0 0 -1.17 rpy=0 0.261799387799149 0, axis 0 0 1, limit lower=-100 upper=100 effort=-1 velocity=10

File: urdf/r2d2.urdf (robot description, URDF)
Before this commit: robot r2d2, 12 links, 11 joints
Links:
- added link carrot; visual mesh filename=package://ecn_mobile_control/urdf/carrot/carrot.dae scale=0.003 0.003 0.003
- added link carrot_disable
Joints:
- added joint carrot: type prismatic, parent carrot_disable, child carrot, origin xyz=0 0 0, axis 1 0 0, limit lower=-100 upper=100 effort=-1 velocity=10
- added joint carrot_disable: type prismatic, parent base_link, child carrot_disable, axis 0 0 1, limit lower=-100 upper=100 effort=-1 velocity=10

Commit message: ROS 2 version

File: urdf/bike.urdf (robot description, URDF)
Before this commit: robot frame, 7 links, 6 joints
Links:
- removed link backWheelLink
- removed link carrot
- removed link carrot_disable
- removed link footprint
- removed link frameLink
- removed link frontWheelLink
- removed link handlebarLink
- added link robot/backWheelLink, mass 1.0; collision mesh filename=package://mobro/urdf/files/wheel_scaled.stl; visual mesh filename=package://mobro/urdf/files/wheel_scaled.stl
- added link robot/base_footprint
- added link robot/carrot; visual mesh filename=package://mobro/urdf/carrot/carrot.dae scale=0.003 0.003 0.003
- added link robot/carrot_disable
- added link robot/frameLink, mass 5.0; collision mesh filename=package://mobro/urdf/files/frame_scaled_left.stl; collision mesh filename=package://mobro/urdf/files/frame_scaled_right.stl
- added link robot/frontWheelLink, mass 1.0; collision mesh filename=package://mobro/urdf/files/wheel_scaled.stl; visual mesh filename=package://mobro/urdf/files/wheel_scaled.stl
- added link robot/handlebarLink, mass .5; collision mesh filename=package://mobro/urdf/files/handlebar_scaled.stl; visual mesh filename=package://mobro/urdf/files/handlebar_scaled.stl
Joints:
- joint carrot: child carrot -> robot/carrot; parent carrot_disable -> robot/carrot_disable
- joint carrot_disable: child carrot_disable -> robot/carrot_disable; parent handlebarLink -> robot/handlebarLink
- joint footprint: child frameLink -> robot/frameLink; parent footprint -> robot/base_footprint
- joint frame_to_backwheel: child backWheelLink -> robot/backWheelLink; parent frameLink -> robot/frameLink
- joint frame_to_handlebar: child handlebarLink -> robot/handlebarLink; limit effort=100 velocity=100 -> lower=-1.57 upper=1.57 effort=100 velocity=100; parent frameLink -> robot/frameLink; type continuous -> revolute
- joint handlebar_to_frontwheel: child frontWheelLink -> robot/frontWheelLink; parent handlebarLink -> robot/handlebarLink

File: urdf/r2d2.urdf (robot description, URDF)
Before this commit: robot r2d2, 14 links, 13 joints
Links:
- removed link base_link
- removed link box
- removed link carrot
- removed link carrot_disable
- removed link footprint
- removed link head
- removed link left_back_wheel
- removed link left_base
- removed link left_front_wheel
- removed link left_leg
- removed link right_back_wheel
- removed link right_base
- removed link right_front_wheel
- removed link right_leg
- added link robot/base_footprint
- added link robot/base_link; visual cylinder length=0.6 radius=0.2
- added link robot/box; visual box size=.08 .08 .08
- added link robot/carrot; visual mesh filename=package://mobro/urdf/carrot/carrot.dae scale=0.003 0.003 0.003
- added link robot/carrot_disable
- added link robot/head; visual sphere radius=0.2
- added link robot/left_back_wheel; visual cylinder length=0.1 radius=0.035
- added link robot/left_base; visual box size=0.4 .1 .1
- added link robot/left_front_wheel; visual cylinder length=0.1 radius=0.035
- added link robot/left_leg; visual box size=0.6 .1 .2
- added link robot/right_back_wheel; visual cylinder length=0.1 radius=0.035
- added link robot/right_base; visual box size=0.4 .1 .1
- added link robot/right_front_wheel; visual cylinder length=0.1 radius=0.035
- added link robot/right_leg; visual box size=0.6 .1 .2
Joints:
- joint base_to_left_leg: child left_leg -> robot/left_leg; parent base_link -> robot/base_link
- joint base_to_right_leg: child right_leg -> robot/right_leg; parent base_link -> robot/base_link
- joint carrot: child carrot -> robot/carrot; parent carrot_disable -> robot/carrot_disable
- joint carrot_disable: child carrot_disable -> robot/carrot_disable; parent footprint -> robot/base_footprint
- joint footprint: child base_link -> robot/base_link; parent footprint -> robot/base_footprint
- joint head_swivel: child head -> robot/head; parent base_link -> robot/base_link
- joint left_back_wheel_joint: child left_back_wheel -> robot/left_back_wheel; parent left_base -> robot/left_base
- joint left_base_joint: child left_base -> robot/left_base; parent left_leg -> robot/left_leg
- joint left_front_wheel_joint: child left_front_wheel -> robot/left_front_wheel; parent left_base -> robot/left_base
- joint right_back_wheel_joint: child right_back_wheel -> robot/right_back_wheel; parent right_base -> robot/right_base
- joint right_base_joint: child right_base -> robot/right_base; parent right_leg -> robot/right_leg
- joint right_front_wheel_joint: child right_front_wheel -> robot/right_front_wheel; parent right_base -> robot/right_base
- joint tobox: child box -> robot/box; parent head -> robot/head
